File: TheSedan.kicad_pcb (KiCad board)
At the start: 2 copper layers, 309.6 x 138.9 mm, 152 parts, among them SW1 SW_Push, U2 ATmega32U4-AU, Y1 16MHz

Commit message: 5/4/20 v3
Parts:
- F1: footprint Fuse:Fuse_1206_3216Metric -> Fuse:Fuse_1210_3225Metric
- USB1: footprint random-keyboard-parts:Molex-0548190589 -> Connector_USB:USB_Micro-B_Molex_47346-0001; moved to B.Cu
- moved F1 75.6 mm to (426.2, 29.4), turned to 180 degrees
- moved U2 69.7 mm to (428.6, 39.7), turned to 270 degrees
- moved SW1 46.5 mm to (415.9, 59.5)
- moved C1 43.9 mm to (401.6, 37.3), turned to 180 degrees
- moved C2 39.0 mm to (401.6, 42.1), turned to 180 degrees
- moved R2 36.1 mm to (408.8, 54.8)
- moved C7 36.0 mm to (401.6, 65.9), turned to 180 degrees
- moved R4 33.3 mm to (408.8, 64.3)
- moved R3 31.2 mm to (408.8, 59.5)
- moved R1 30.8 mm to (408.8, 50.0)
- moved C6 27.8 mm to (401.6, 61.1), turned to 180 degrees
- moved C5 25.9 mm to (401.6, 56.4), turned to 180 degrees
- moved C4 25.4 mm to (401.6, 51.6), turned to 180 degrees
- moved C3 20.7 mm to (401.6, 46.8), turned to 180 degrees
- moved Y1 11.7 mm to (415.1, 41.3), turned to 90 degrees
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Connections:
- U2 pad 10: col12 -> Net-(U2-Pad10)
- U2 pad 11: col11 -> Net-(U2-Pad11)
- U2 pad 12: col7 -> col0
- U2 pad 18: col2 -> col1
- U2 pad 19: col1 -> col2
- U2 pad 20: col0 -> col3
- U2 pad 21: col6 -> col4
- U2 pad 22: Net-(U2-Pad22) -> col5
- U2 pad 25: col3 -> col6
- U2 pad 26: Net-(U2-Pad26) -> col7
- U2 pad 27: Net-(U2-Pad27) -> col8
- U2 pad 28: col10 -> col9
- U2 pad 29: col9 -> col10
- U2 pad 30: col8 -> col11
- U2 pad 31: col5 -> col12
- U2 pad 32: col4 -> col13
- U2 pad 36: row0 -> col14
- U2 pad 37: row1 -> row0
- U2 pad 38: row2 -> row1
- U2 pad 39: row3 -> row2
- U2 pad 40: row4 -> row3
- U2 pad 41: Net-(U2-Pad41) -> row4
- U2 pad 8: col14 -> Net-(U2-Pad8)
- U2 pad 9: col13 -> Net-(U2-Pad9)
Routing:
- net GND: track 0.00 -> 125.9 mm, vias 0 -> 3
- net +5V: track 0.00 -> 93.0 mm, vias 0 -> 4
- net Net-(D54-Pad2): track 70.4 -> 144.3 mm
- net Net-(D58-Pad2): track 89.1 -> 160.1 mm
- net Net-(D53-Pad2): track 43.3 -> 104.9 mm
- net Net-(D55-Pad2): track 98.3 -> 156.3 mm
- net Net-(R1-Pad1): track 0.00 -> 56.4 mm, vias 0 -> 2
- net Net-(C3-Pad1): track 0.00 -> 47.7 mm, vias 0 -> 2
- net Net-(D52-Pad2): track 21.4 -> 69.0 mm
- net Net-(D45-Pad2): track 108.4 -> 154.0 mm
- net Net-(R4-Pad2): track 0.00 -> 41.0 mm, vias 0 -> 2
- net Net-(R2-Pad1): track 0.00 -> 40.9 mm, vias 0 -> 2
- net col0: track 103.2 -> 142.9 mm, vias 0 -> 2
- net Net-(D44-Pad2): track 99.0 -> 133.1 mm
- net Net-(D57-Pad2): track 33.5 -> 66.3 mm
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Other:
- board text added: "The Sedan"
- board text added: "rev2.0"

Commit message: 5/4/20 v3
Parts:
- C1, C2, C3, C4, C5, C6, C7, D1, D10, D11, D12, D13, D14, D15, D16, D17, D18, D19, D2, D20, D21, D22, D23, D24, D25, D26, D27, D28, D29, D3, D30, D31, D32, D33, D34, D35, D36, D37, D38, D39, D4, D40, D41, D42, D43, D44, D45, D46, D47, D48, D49, D5, D50, D51, D52, D53, D54, D55, D56, D57, D58, D59, D6, D60, D61, D62, D63, D64, D65, D66, D67, D68, D7, D8, D9, F1, R1, R2, R3, R4, SW1, U2, Y1: moved to B.Cu
- moved C4 155.4 mm to (514.2, 158.8), turned to 45 degrees
- moved C5 149.9 mm to (511.2, 158.8), turned to 45 degrees
- moved R1 148.7 mm to (505.8, 162.7)
- moved C3 147.9 mm to (493.6, 162.7), turned to 0 degrees
- moved C6 144.4 mm to (508.0, 158.8), turned to 45 degrees
- moved R2 141.8 mm to (500.7, 162.7)
- moved D5 139.5 mm to (403.3, 161.1), turned to 0 degrees
- moved C7 138.8 mm to (504.8, 158.8), turned to 45 degrees
- moved C1 137.7 mm to (481.8, 149.2)
- moved R4 137.0 mm to (517.5, 147.6), turned to 90 degrees
- moved D10 135.6 mm to (427.1, 161.1), turned to 0 degrees
- moved C2 134.2 mm to (477.0, 153.1), turned to 90 degrees
- moved D15 132.5 mm to (450.9, 161.1), turned to 0 degrees
- moved U2 131.4 mm to (496.1, 152.4), turned to 90 degrees
- moved Y1 130.0 mm to (481.8, 152.9), turned to 270 degrees
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Routing:
- net Net-(D6-Pad2): track 325.8 -> 11.4 mm, vias 1 -> 0
- net Net-(D7-Pad2): track 325.2 -> 11.4 mm, vias 1 -> 0
- net Net-(D8-Pad2): track 315.4 -> 11.4 mm, vias 1 -> 0
- net Net-(D9-Pad2): track 308.4 -> 11.4 mm, vias 1 -> 0
- net Net-(D10-Pad2): track 286.2 -> 11.4 mm, vias 1 -> 0
- net col13: track 328.9 -> 82.2 mm
- net col12: track 304.0 -> 83.6 mm
- net col11: track 291.0 -> 90.7 mm
- net col10: track 268.1 -> 83.3 mm
- net Net-(D15-Pad2): track 189.1 -> 11.4 mm, vias 1 -> 0
- net Net-(D5-Pad2): track 181.6 -> 11.4 mm, vias 1 -> 0
- net col9: track 248.8 -> 83.3 mm
- net col14: track 351.4 -> 189.6 mm
- net Net-(D32-Pad2): track 165.8 -> 11.4 mm, vias 1 -> 0
- net Net-(D14-Pad2): track 164.2 -> 11.4 mm, vias 1 -> 0
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Other:
- board outline removed
- board text added: "rev2.1"
- board text removed: "rev2.0"

Commit message: 5/5/20 v1
Parts:
- moved SW1 14.3 mm to (467.5, 73.0)
- moved R4 7.69 mm to (514.4, 154.6), turned to 135 degrees
Connections:
- U2 pad 21: col4 -> row0
- U2 pad 22: col5 -> row2
- U2 pad 25: col6 -> row1
- U2 pad 26: col7 -> col5
- U2 pad 27: col8 -> col4
- U2 pad 28: col9 -> row3
- U2 pad 29: col10 -> col7
- U2 pad 30: col11 -> col8
- U2 pad 31: col12 -> col9
- U2 pad 32: col13 -> col10
- U2 pad 36: col14 -> col11
- U2 pad 37: row0 -> col12
- U2 pad 38: row1 -> col13
- U2 pad 39: row2 -> col14
- U2 pad 40: row3 -> col6
Routing:
- net col13: track 82.2 -> 251.2 mm, vias 0 -> 1
- net D+: track 2.51 -> 161.4 mm, vias 1 -> 4
- net D-: track 3.36 -> 156.0 mm, vias 1 -> 4
- net col12: track 83.6 -> 236.1 mm, vias 0 -> 1
- net col11: track 90.7 -> 227.1 mm, vias 0 -> 1
- net col10: track 83.3 -> 201.8 mm, vias 0 -> 1
- net col9: track 83.3 -> 183.7 mm, vias 0 -> 1
- net col8: track 64.3 -> 163.3 mm, vias 0 -> 1
- net col14: track 189.6 -> 269.9 mm, vias 0 -> 1
- net col7: track 64.3 -> 144.3 mm, vias 0 -> 1
- net GND: track 108.8 -> 185.8 mm, vias 4 -> 6
- net row0: track 303.4 -> 378.2 mm, vias 0 -> 6
- net VCC: track 4.22 -> 73.4 mm, vias 1 -> 4
- net row1: track 298.6 -> 344.7 mm, vias 0 -> 2
- net col5: track 64.3 -> 94.3 mm, vias 0 -> 1
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- added copper zone on B.Cu, net GND
